File: PCB/kraky2.kicad_pcb (KiCad board)
At the start: 2 copper layers, 95 x 95.8 mm, 127 parts, among them J1 CQ-USB-C16PSMT01, J2 PINHD_1x8_Female, J3 JST_02, J4 142-0701-501, J5 142-0701-501, J6 MSD-4-A, J7 U.FL-R-SMT_01_, Q1 2N3904, Q2 BC107, Q3 BC107, Q4 BC107, Q5 BC107, SW1 Push_Button, SW2 Push_Button, SW3 Push_Button, SW4 Push_Button, SW5 SW_Nidec_CAS-120A1, SW6 RESET, SW7 BOOT, U1 AMS1117-3.3, U10 MFRC522, U11 ESP32-S3-WROOM-1, U3 CH343P, U4 CN3063-SOIC8, U5 NRF24L01, U6 PN5321A3HN_C1xx, U8 CC1101, U9 TPS61023DRLR, Y1 16 MHz, Y2 26 MHz, Y3 27.12 MHz, Y4 27.12 MHz

Commit message: Add files via upload
Parts:
- added R25: 100K, Resistor_SMD:R_0805_2012Metric, F.Cu at (118.5, 145.8)
- added R26: 100K, Resistor_SMD:R_0805_2012Metric, F.Cu at (115.2, 145.8)
- L11, L12: footprint Inductor_SMD:L_0805_2012Metric -> Inductor_SMD:L_1206_3216Metric_Pad1.22x1.90mm_HandSolder
- L14, L15: footprint Inductor_SMD:L_0805_2012Metric -> CD54:IND_CD54_SUM
- moved C44 3.50 mm to (151.8, 104.7)
- moved C42 3.45 mm to (156.2, 108.5)
- moved C43 3.45 mm to (156.2, 101.0)
- moved C45 3.45 mm to (156.2, 104.5)
- moved C46 3.45 mm to (160.2, 104.5)
- moved C47 3.45 mm to (164.2, 104.5)
- moved R15 3.45 mm to (162.7, 108.5)
- moved R18 3.45 mm to (162.7, 101.0)
- moved L15 2.47 mm to (150.2, 108.8)
- moved L14 2.10 mm to (150.3, 100.5)
- moved C31 1.29 mm to (162.2, 81.5)
- moved C36 1.29 mm to (165.7, 81.6)
- moved C33 1.01 mm to (162.2, 85.0)
- moved C34 1.01 mm to (161.9, 87.2)
- moved C35 1.01 mm to (165.4, 86.5)
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Connections:
- U11 pad 17: unconnected-(U11-IO9-Pad17) -> BATT
Routing:
- net BATT: track 0.00 -> 29.0 mm, vias 0 -> 4
- net Net-(D5-A): track 98.3 -> 108.9 mm
- net Net-(Q4-E): track 3.46 -> 6.34 mm
- net 3V3: track 430.2 -> 432.7 mm
- net RFANT1: track 34.1 -> 31.9 mm
- net RFANT2: track 20.0 -> 18.2 mm
- net Net-(Q5-E): track 3.95 -> 5.68 mm
- net GND: track 319.5 -> 321.0 mm, vias 506 -> 507
- net Net-(C43-Pad1): track 6.82 -> 8.08 mm
- net Net-(C31-Pad1): track 5.00 -> 5.60 mm

Commit message: Add files via upload
Connections:
- J2 pad 5: RST -> RST A
- U11 pad 18: unconnected-(U11-IO10-Pad18) -> RST A
Routing:
- net RST: track 45.6 -> 2.25 mm, vias 2 -> 0
- net RST A: track 0.00 -> 39.5 mm, vias 0 -> 2
- net DC A: track 35.2 -> 35.3 mm, vias 2 -> 4
- net SCK: vias 8 -> 10
